File: RX.sch (EAGLE design)
At the start: 35 parts, among them IC1 OPA354AIDBVR, IC2 LM7171BIN_NOPB, IC3 LTC6268IS6-10#TRMPBF, U1 OPA656U, X1 BU-SMA-V

Commit message: memberikan komponen kompnen yang dibutukan pada rangkaian TIA dengan IC LTC6268 kecuali filter untuk HPF
Parts:
- added BIAS_CONN, SUPPLY-TIA+, SUPPLY-TIA-: 455-1750-1-ND, SparkFun-Connectors:CONN_03
- added C11, C14, C15, C16, C17, C18, C22, C24: 06033C104KAZ2A, SamacSys_Parts:06033C104KAZ2A
- added C19, C21, C23, C25: 10uF, SparkFun-Capacitors:10UF-POLAR-0603-6.3V-20%(TANT)
- added D6, D7, D8, D9: BPV10NF, SamacSys_Parts:BPV10NF
- added IC4: TPS72325DBVTG4, SamacSys_Parts:TPS72325DBVTG4
- added IC5: TLV75525PDBVR, SamacSys_Parts:TLV75525PDBVR
- added IC6: TC7662BEOA, SamacSys_Parts:TC7662BEOA
- added INPUT, OUTPUT_LTC: (no value), SparkFun-Connectors:CONN_02
- added JP5: JUMPER-SMT_2_NC_TRACE_NO-SILK, SparkFun-Jumpers:JUMPER-SMT_2_NC_TRACE_NO-SILK
- added R7: RG2012P-275-B-T5, SamacSys_Parts:RG2012P-275-B-T5
- J4: value (none) -> 455-1750-1-ND
Connections:
- new net +2.5V: BIAS_CONN.1, C18.2, IC5.OUT, SUPPLY-TIA+.3
- new net +5V: C17.2, C21.+, C22.2, IC5.EN, IC5.IN, IC6.V+, INPUT.1, SUPPLY-TIA+.1
- new net -2.5V: C15.2, IC4.OUT, SUPPLY-TIA-.1
- new net FILTER_IN: JP5.2
- new net GND2: BIAS_CONN.3, C14.1, C15.1, C16.1, C17.1, C18.1, C19.+, C21.-, C22.1, C23.+, C24.1, IC3.IN+, IC4.GND, IC6.GND, INPUT.2, OUTPUT_LTC.1, SUPPLY-TIA-.3
- new net N$10: C11.1, IC3.OUT, JP5.1, OUTPUT_LTC.2, R7.1
- new net N$11: C25.+, IC6.CAP+
- new net N$12: C25.-, IC6.CAP-
- new net N$13: D6.K, D7.K, D8.K, D9.K
- new net N$14: C11.2, D6.A, D7.A, D8.A, D9.A, IC3.-IN, R7.2
- new net N$9: C16.2, IC4.NR/FB
- new net V+: IC3.V+, SUPPLY-TIA+.2
- new net V-: IC3.V-, SUPPLY-TIA-.2
- new net V_BIAS: BIAS_CONN.2
- net -5V: now also C14.2, C19.-, C23.-, C24.2, IC4.EN, IC4.IN, IC6.VOUT

Commit message: Menambahakan komponen komponen yang diperlukan untuk OPA656U kurang HPF untuk rangkaian OPA656U
Parts:
- removed U1: OPA656U, Texas Instruments_By_element14_Batch_1:OPA656U
- added C20, C26, C27, C31, C33: 06033C104KAZ2A, SamacSys_Parts:06033C104KAZ2A
- added C28, C29, C30, C32: 10uF, SparkFun-Capacitors:10UF-POLAR-0603-6.3V-20%(TANT)
- added D10, D11, D12, D13: VBPW34SR, SamacSys_Parts:VBPW34SR
- added IC7: OPA656U, SamacSys_Parts:OPA656U
- added IC8: TC7662BEOA, SamacSys_Parts:TC7662BEOA
- added INPUT656U, OUT656U: (no value), SparkFun-Connectors:CONN_02
- added JP6: JUMPER-SMT_2_NC_TRACE_NO-SILK, SparkFun-Jumpers:JUMPER-SMT_2_NC_TRACE_NO-SILK
- added R8: RG2012P-275-B-T5, SamacSys_Parts:RG2012P-275-B-T5
Connections:
- new net +V656U: C32.+, C33.2, IC7.+VS, IC8.V+, INPUT656U.1
- new net -5VLTC: C14.2, C19.-, C23.-, C24.2, IC4.EN, IC4.IN, IC6.VOUT
- new net -V656U: C29.-, C30.-, C31.2, IC7.-VS, IC8.VOUT
- new net GND3: C26.1, C27.1, C29.+, C30.+, C31.1, C32.-, C33.1, IC7.NON-INVERTING_INPUT, IC8.GND, INPUT656U.2, OUT656U.2
- new net N$15: C28.+, IC8.CAP+
- new net N$17: C28.-, IC8.CAP-
- new net N$2: C20.1, C26.2, C27.2, D10.A, D11.A, D12.A, D13.A, IC7.INVERTING_INPUT, R8.1
- new net V_BIAS656U: D10.K, D11.K, D12.K, D13.K
- net -5V: no longer C14.2, C19.-, C23.-, C24.2, IC4.EN, IC4.IN, IC6.VOUT
- net GND2: now also IC5.GND
- net N$13: now also C20.2, IC7.OUTPUT, JP6.1, OUT656U.1, R8.2; no longer D6.K, D7.K, D8.K, D9.K
- net V_BIAS: now also D6.K, D7.K, D8.K, D9.K
