File: RX.brd (EAGLE design)
At the start: 160 x 100 mm, 61 parts, among them IC1 OPA354AIDBVR, IC2 LM7171BIN_NOPB, IC3 LTC6268IS6-10#TRMPBF, IC4 TPS72325DBVTG4, IC5 TLV75525PDBVR, IC6 TC7662BEOA, J4 455-1750-1-ND, U1 OPA656U, X1 BU-SMA-V

Commit message: melakukan routing untuk sheet 2 , belum ada filter
Parts:
- moved OUTPUT_LTC 168.7 mm to (41.7, 23.7), flipped to the bottom
- moved BIAS_CONN 151.7 mm to (36.6, 20.2)
- moved C19 144.5 mm to (16.3, 9.02), turned to 180 degrees
- moved C25 139.7 mm to (9.59, 12.4), turned to 90 degrees
- moved JP5 130.9 mm to (36.5, 23.7), turned to 180 degrees
- moved C21 126.8 mm to (26.6, 16.4)
- moved C22 126.2 mm to (26.7, 14.6)
- moved C24 124.5 mm to (19.5, 7.95), turned to 90 degrees
- moved SUPPLY-TIA+ 124.2 mm to (28.5, 20.2)
- moved C23 119.8 mm to (16.3, 7.03), turned to 180 degrees
- moved SUPPLY-TIA- 117.9 mm to (26.7, 7.17)
- moved INPUT 116.4 mm to (25.5, 20.2), turned to 180 degrees
- moved D9 104.9 mm to (47.6, 10.6), turned to 90 degrees
- moved R7 99.7 mm to (42.8, 10.2), turned to 90 degrees
- moved D8 86.1 mm to (47.6, 17.9), turned to 270 degrees
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Connections:
- removed net N$13: D6.1, D7.1, D8.1, D9.1
- new net -5V_LTC: C14.2, C19.-, C23.-, C24.2, IC4.2, IC4.3, IC6.5
- net -5V: no longer C14.2, C19.-, C23.-, C24.2, IC4.2, IC4.3, IC6.5
- net GND: no longer IC5.2
- net GND2: now also IC5.2
- net V_BIAS: now also D6.1, D7.1, D8.1, D9.1
Routing:
- net GND2: track 0.00 -> 133.5 mm
- net V_BIAS: track 0.00 -> 45.1 mm
- net +5V: track 0.00 -> 33.6 mm
- net N$10: track 0.00 -> 33.1 mm
- net N$14: track 0.00 -> 30.1 mm
- net -2.5V: track 0.00 -> 24.5 mm, vias 0 -> 2
- net V+: track 0.00 -> 19.0 mm, vias 0 -> 2
- net V-: track 0.00 -> 14.9 mm, vias 0 -> 2
- net +2.5V: track 0.00 -> 14.7 mm
- net -5V_LTC: track 0.00 -> 11.6 mm
- net N$12: track 0.00 -> 3.16 mm
- net N$11: track 0.00 -> 2.81 mm
- net N$9: track 0.00 -> 1.77 mm
- added copper zone on layer 1, net GND2
- added copper zone on layer 1, net LTC6268
